File: kp_gmapminiproto.kicad_pcb (KiCad board)
At the start: 10 copper layers, 416.6 x 152.4 mm, 114 parts, among them SW00_00 SW, SW00_01 SW, SW00_02 SW, SW00_03 SW, SW01_00 SW, SW01_01 SW, SW01_02 SW, SW01_03 SW, SW02_00 SW, SW02_01 SW, SW02_02 SW, SW02_03 SW, SW03_00 SW, SW03_01 SW, SW03_02 SW, SW03_03 SW

Commit message: update for kicad 7
Connections:
- D_IC_02 pad 10: (no net) -> unconnected-(D_IC_02-~{OUT5}-Pad10)
- D_IC_02 pad 11: (no net) -> unconnected-(D_IC_02-~{OUT6}-Pad11)
- D_IC_02 pad 12: (no net) -> unconnected-(D_IC_02-~{OUT7}-Pad12)
- D_IC_02 pad 5: (no net) -> unconnected-(D_IC_02-~{OUT0}-Pad5)
- D_IC_02 pad 6: (no net) -> unconnected-(D_IC_02-~{OUT1}-Pad6)
- D_IC_02 pad 7: (no net) -> unconnected-(D_IC_02-~{OUT2}-Pad7)
- D_IC_02 pad 8: (no net) -> unconnected-(D_IC_02-~{OUT3}-Pad8)
- D_IC_02 pad 9: (no net) -> unconnected-(D_IC_02-~{OUT4}-Pad9)
- D_IC_03 pad 10: (no net) -> unconnected-(D_IC_03-~{OUT5}-Pad10)
- D_IC_03 pad 11: (no net) -> unconnected-(D_IC_03-~{OUT6}-Pad11)
- D_IC_03 pad 12: (no net) -> unconnected-(D_IC_03-~{OUT7}-Pad12)
- D_IC_03 pad 5: (no net) -> unconnected-(D_IC_03-~{OUT0}-Pad5)
- D_IC_03 pad 6: (no net) -> unconnected-(D_IC_03-~{OUT1}-Pad6)
- D_IC_03 pad 7: (no net) -> unconnected-(D_IC_03-~{OUT2}-Pad7)
- D_IC_03 pad 8: (no net) -> unconnected-(D_IC_03-~{OUT3}-Pad8)
- D_IC_03 pad 9: (no net) -> unconnected-(D_IC_03-~{OUT4}-Pad9)
- D_IC_04 pad 10: (no net) -> unconnected-(D_IC_04-~{OUT5}-Pad10)
- D_IC_04 pad 11: (no net) -> unconnected-(D_IC_04-~{OUT6}-Pad11)
- D_IC_04 pad 12: (no net) -> unconnected-(D_IC_04-~{OUT7}-Pad12)
- D_IC_04 pad 5: (no net) -> unconnected-(D_IC_04-~{OUT0}-Pad5)
- D_IC_04 pad 6: (no net) -> unconnected-(D_IC_04-~{OUT1}-Pad6)
- D_IC_04 pad 7: (no net) -> unconnected-(D_IC_04-~{OUT2}-Pad7)
- D_IC_04 pad 8: (no net) -> unconnected-(D_IC_04-~{OUT3}-Pad8)
- D_IC_04 pad 9: (no net) -> unconnected-(D_IC_04-~{OUT4}-Pad9)
- D_IC_05 pad 10: (no net) -> unconnected-(D_IC_05-~{OUT5}-Pad10)
- D_IC_05 pad 11: (no net) -> unconnected-(D_IC_05-~{OUT6}-Pad11)
- D_IC_05 pad 12: (no net) -> unconnected-(D_IC_05-~{OUT7}-Pad12)
- D_IC_05 pad 5: (no net) -> unconnected-(D_IC_05-~{OUT0}-Pad5)
- D_IC_05 pad 6: (no net) -> unconnected-(D_IC_05-~{OUT1}-Pad6)
- D_IC_05 pad 7: (no net) -> unconnected-(D_IC_05-~{OUT2}-Pad7)
- D_IC_05 pad 8: (no net) -> unconnected-(D_IC_05-~{OUT3}-Pad8)
- D_IC_05 pad 9: (no net) -> unconnected-(D_IC_05-~{OUT4}-Pad9)
- D_IC_06 pad 10: (no net) -> unconnected-(D_IC_06-~{OUT5}-Pad10)
- D_IC_06 pad 11: (no net) -> unconnected-(D_IC_06-~{OUT6}-Pad11)
- D_IC_06 pad 12: (no net) -> unconnected-(D_IC_06-~{OUT7}-Pad12)
- D_IC_06 pad 5: (no net) -> unconnected-(D_IC_06-~{OUT0}-Pad5)
- D_IC_06 pad 6: (no net) -> unconnected-(D_IC_06-~{OUT1}-Pad6)
- D_IC_06 pad 7: (no net) -> unconnected-(D_IC_06-~{OUT2}-Pad7)
- D_IC_06 pad 8: (no net) -> unconnected-(D_IC_06-~{OUT3}-Pad8)
- D_IC_06 pad 9: (no net) -> unconnected-(D_IC_06-~{OUT4}-Pad9)
- D_IC_07 pad 10: (no net) -> unconnected-(D_IC_07-~{OUT5}-Pad10)
- D_IC_07 pad 11: (no net) -> unconnected-(D_IC_07-~{OUT6}-Pad11)
- D_IC_07 pad 12: (no net) -> unconnected-(D_IC_07-~{OUT7}-Pad12)
- D_IC_07 pad 14: (no net) -> unconnected-(D_IC_07-SDO-Pad14)
- D_IC_07 pad 5: (no net) -> unconnected-(D_IC_07-~{OUT0}-Pad5)
- D_IC_07 pad 6: (no net) -> unconnected-(D_IC_07-~{OUT1}-Pad6)
- D_IC_07 pad 7: (no net) -> unconnected-(D_IC_07-~{OUT2}-Pad7)
- D_IC_07 pad 8: (no net) -> unconnected-(D_IC_07-~{OUT3}-Pad8)
- D_IC_07 pad 9: (no net) -> unconnected-(D_IC_07-~{OUT4}-Pad9)
- RV_IC_02 pad 1: (no net) -> unconnected-(RV_IC_02-CH0-Pad1)
- RV_IC_02 pad 2: (no net) -> unconnected-(RV_IC_02-CH1-Pad2)
- RV_IC_02 pad 3: (no net) -> unconnected-(RV_IC_02-CH2-Pad3)
- RV_IC_02 pad 4: (no net) -> unconnected-(RV_IC_02-CH3-Pad4)
- RV_IC_02 pad 5: (no net) -> unconnected-(RV_IC_02-CH4-Pad5)
- RV_IC_02 pad 6: (no net) -> unconnected-(RV_IC_02-CH5-Pad6)
- RV_IC_02 pad 7: (no net) -> unconnected-(RV_IC_02-CH6-Pad7)
- RV_IC_02 pad 8: (no net) -> unconnected-(RV_IC_02-CH7-Pad8)
- RV_IC_03 pad 1: (no net) -> unconnected-(RV_IC_03-CH0-Pad1)
- RV_IC_03 pad 2: (no net) -> unconnected-(RV_IC_03-CH1-Pad2)
- RV_IC_03 pad 3: (no net) -> unconnected-(RV_IC_03-CH2-Pad3)
- RV_IC_03 pad 4: (no net) -> unconnected-(RV_IC_03-CH3-Pad4)
- RV_IC_03 pad 5: (no net) -> unconnected-(RV_IC_03-CH4-Pad5)
- RV_IC_03 pad 6: (no net) -> unconnected-(RV_IC_03-CH5-Pad6)
- RV_IC_03 pad 7: (no net) -> unconnected-(RV_IC_03-CH6-Pad7)
- RV_IC_03 pad 8: (no net) -> unconnected-(RV_IC_03-CH7-Pad8)
- RV_IC_04 pad 1: (no net) -> unconnected-(RV_IC_04-CH0-Pad1)
- RV_IC_04 pad 2: (no net) -> unconnected-(RV_IC_04-CH1-Pad2)
- RV_IC_04 pad 3: (no net) -> unconnected-(RV_IC_04-CH2-Pad3)
- RV_IC_04 pad 4: (no net) -> unconnected-(RV_IC_04-CH3-Pad4)
- RV_IC_04 pad 5: (no net) -> unconnected-(RV_IC_04-CH4-Pad5)
- RV_IC_04 pad 6: (no net) -> unconnected-(RV_IC_04-CH5-Pad6)
- RV_IC_04 pad 7: (no net) -> unconnected-(RV_IC_04-CH6-Pad7)
- RV_IC_04 pad 8: (no net) -> unconnected-(RV_IC_04-CH7-Pad8)
- RV_IC_05 pad 1: (no net) -> unconnected-(RV_IC_05-CH0-Pad1)
- RV_IC_05 pad 2: (no net) -> unconnected-(RV_IC_05-CH1-Pad2)
- RV_IC_05 pad 3: (no net) -> unconnected-(RV_IC_05-CH2-Pad3)
- RV_IC_05 pad 4: (no net) -> unconnected-(RV_IC_05-CH3-Pad4)
- RV_IC_05 pad 5: (no net) -> unconnected-(RV_IC_05-CH4-Pad5)
- RV_IC_05 pad 6: (no net) -> unconnected-(RV_IC_05-CH5-Pad6)
- RV_IC_05 pad 7: (no net) -> unconnected-(RV_IC_05-CH6-Pad7)
- RV_IC_05 pad 8: (no net) -> unconnected-(RV_IC_05-CH7-Pad8)
- RV_IC_06 pad 1: (no net) -> unconnected-(RV_IC_06-CH0-Pad1)
- RV_IC_06 pad 2: (no net) -> unconnected-(RV_IC_06-CH1-Pad2)
- RV_IC_06 pad 3: (no net) -> unconnected-(RV_IC_06-CH2-Pad3)
- RV_IC_06 pad 4: (no net) -> unconnected-(RV_IC_06-CH3-Pad4)
- RV_IC_06 pad 5: (no net) -> unconnected-(RV_IC_06-CH4-Pad5)
- RV_IC_06 pad 6: (no net) -> unconnected-(RV_IC_06-CH5-Pad6)
- RV_IC_06 pad 7: (no net) -> unconnected-(RV_IC_06-CH6-Pad7)
- RV_IC_06 pad 8: (no net) -> unconnected-(RV_IC_06-CH7-Pad8)
- RV_IC_07 pad 1: (no net) -> unconnected-(RV_IC_07-CH0-Pad1)
- RV_IC_07 pad 2: (no net) -> unconnected-(RV_IC_07-CH1-Pad2)
- RV_IC_07 pad 3: (no net) -> unconnected-(RV_IC_07-CH2-Pad3)
- RV_IC_07 pad 4: (no net) -> unconnected-(RV_IC_07-CH3-Pad4)
- RV_IC_07 pad 5: (no net) -> unconnected-(RV_IC_07-CH4-Pad5)
- RV_IC_07 pad 6: (no net) -> unconnected-(RV_IC_07-CH5-Pad6)
- RV_IC_07 pad 7: (no net) -> unconnected-(RV_IC_07-CH6-Pad7)
- RV_IC_07 pad 8: (no net) -> unconnected-(RV_IC_07-CH7-Pad8)
- SW_IC_00 pad 19: (no net) -> unconnected-(SW_IC_00-INTB-Pad19)
- SW_IC_00 pad 20: (no net) -> unconnected-(SW_IC_00-INTA-Pad20)
- SW_IC_01 pad 1: (no net) -> unconnected-(SW_IC_01-GPB0-Pad1)
- SW_IC_01 pad 19: (no net) -> unconnected-(SW_IC_01-INTB-Pad19)
- SW_IC_01 pad 2: (no net) -> unconnected-(SW_IC_01-GPB1-Pad2)
- SW_IC_01 pad 20: (no net) -> unconnected-(SW_IC_01-INTA-Pad20)
- SW_IC_01 pad 21: (no net) -> unconnected-(SW_IC_01-GPA0-Pad21)
- SW_IC_01 pad 22: (no net) -> unconnected-(SW_IC_01-GPA1-Pad22)
- SW_IC_01 pad 23: (no net) -> unconnected-(SW_IC_01-GPA2-Pad23)
- SW_IC_01 pad 24: (no net) -> unconnected-(SW_IC_01-GPA3-Pad24)
- SW_IC_01 pad 25: (no net) -> unconnected-(SW_IC_01-GPA4-Pad25)
- SW_IC_01 pad 26: (no net) -> unconnected-(SW_IC_01-GPA5-Pad26)
- SW_IC_01 pad 27: (no net) -> unconnected-(SW_IC_01-GPA6-Pad27)
- SW_IC_01 pad 28: (no net) -> unconnected-(SW_IC_01-GPA7-Pad28)
- SW_IC_01 pad 3: (no net) -> unconnected-(SW_IC_01-GPB2-Pad3)
- SW_IC_01 pad 4: (no net) -> unconnected-(SW_IC_01-GPB3-Pad4)
- SW_IC_01 pad 5: (no net) -> unconnected-(SW_IC_01-GPB4-Pad5)
- SW_IC_01 pad 6: (no net) -> unconnected-(SW_IC_01-GPB5-Pad6)
- SW_IC_01 pad 7: (no net) -> unconnected-(SW_IC_01-GPB6-Pad7)
- SW_IC_01 pad 8: (no net) -> unconnected-(SW_IC_01-GPB7-Pad8)
- SW_IC_02 pad 1: (no net) -> unconnected-(SW_IC_02-GPB0-Pad1)
- SW_IC_02 pad 19: (no net) -> unconnected-(SW_IC_02-INTB-Pad19)
- SW_IC_02 pad 2: (no net) -> unconnected-(SW_IC_02-GPB1-Pad2)
- SW_IC_02 pad 20: (no net) -> unconnected-(SW_IC_02-INTA-Pad20)
- SW_IC_02 pad 21: (no net) -> unconnected-(SW_IC_02-GPA0-Pad21)
- SW_IC_02 pad 22: (no net) -> unconnected-(SW_IC_02-GPA1-Pad22)
- SW_IC_02 pad 23: (no net) -> unconnected-(SW_IC_02-GPA2-Pad23)
- SW_IC_02 pad 24: (no net) -> unconnected-(SW_IC_02-GPA3-Pad24)
- SW_IC_02 pad 25: (no net) -> unconnected-(SW_IC_02-GPA4-Pad25)
- SW_IC_02 pad 26: (no net) -> unconnected-(SW_IC_02-GPA5-Pad26)
- SW_IC_02 pad 27: (no net) -> unconnected-(SW_IC_02-GPA6-Pad27)
- SW_IC_02 pad 28: (no net) -> unconnected-(SW_IC_02-GPA7-Pad28)
- SW_IC_02 pad 3: (no net) -> unconnected-(SW_IC_02-GPB2-Pad3)
- SW_IC_02 pad 4: (no net) -> unconnected-(SW_IC_02-GPB3-Pad4)
- SW_IC_02 pad 5: (no net) -> unconnected-(SW_IC_02-GPB4-Pad5)
- SW_IC_02 pad 6: (no net) -> unconnected-(SW_IC_02-GPB5-Pad6)
- SW_IC_02 pad 7: (no net) -> unconnected-(SW_IC_02-GPB6-Pad7)
- SW_IC_02 pad 8: (no net) -> unconnected-(SW_IC_02-GPB7-Pad8)
- SW_IC_03 pad 1: (no net) -> unconnected-(SW_IC_03-GPB0-Pad1)
- SW_IC_03 pad 19: (no net) -> unconnected-(SW_IC_03-INTB-Pad19)
- SW_IC_03 pad 2: (no net) -> unconnected-(SW_IC_03-GPB1-Pad2)
- SW_IC_03 pad 20: (no net) -> unconnected-(SW_IC_03-INTA-Pad20)
- SW_IC_03 pad 21: (no net) -> unconnected-(SW_IC_03-GPA0-Pad21)
- SW_IC_03 pad 22: (no net) -> unconnected-(SW_IC_03-GPA1-Pad22)
- SW_IC_03 pad 23: (no net) -> unconnected-(SW_IC_03-GPA2-Pad23)
- SW_IC_03 pad 24: (no net) -> unconnected-(SW_IC_03-GPA3-Pad24)
- SW_IC_03 pad 25: (no net) -> unconnected-(SW_IC_03-GPA4-Pad25)
- SW_IC_03 pad 26: (no net) -> unconnected-(SW_IC_03-GPA5-Pad26)
- SW_IC_03 pad 27: (no net) -> unconnected-(SW_IC_03-GPA6-Pad27)
- SW_IC_03 pad 28: (no net) -> unconnected-(SW_IC_03-GPA7-Pad28)
- SW_IC_03 pad 3: (no net) -> unconnected-(SW_IC_03-GPB2-Pad3)
- SW_IC_03 pad 4: (no net) -> unconnected-(SW_IC_03-GPB3-Pad4)
- SW_IC_03 pad 5: (no net) -> unconnected-(SW_IC_03-GPB4-Pad5)
- SW_IC_03 pad 6: (no net) -> unconnected-(SW_IC_03-GPB5-Pad6)
- SW_IC_03 pad 7: (no net) -> unconnected-(SW_IC_03-GPB6-Pad7)
- SW_IC_03 pad 8: (no net) -> unconnected-(SW_IC_03-GPB7-Pad8)
- TEENSY_00 pad 15: (no net) -> unconnected-(TEENSY_00-VBAT-Pad15)
- TEENSY_00 pad 16: (no net) -> unconnected-(TEENSY_00-3V3-Pad16)
- TEENSY_00 pad 17: (no net) -> unconnected-(TEENSY_00-GND-Pad17)
- TEENSY_00 pad 18: (no net) -> unconnected-(TEENSY_00-PROGRAM-Pad18)
- TEENSY_00 pad 19: (no net) -> unconnected-(TEENSY_00-ON_OFF-Pad19)
- TEENSY_00 pad 2: (no net) -> unconnected-(TEENSY_00-0_RX1_CRX2_CS1-Pad2)
- TEENSY_00 pad 21: (no net) -> unconnected-(TEENSY_00-14_A0_TX3_SPDIF_OUT-Pad21)
- TEENSY_00 pad 22: (no net) -> unconnected-(TEENSY_00-15_A1_RX3_SPDIF_IN-Pad22)
- TEENSY_00 pad 23: (no net) -> unconnected-(TEENSY_00-16_A2_RX4_SCL1-Pad23)
- TEENSY_00 pad 24: (no net) -> unconnected-(TEENSY_00-17_A3_TX4_SDA1-Pad24)
- TEENSY_00 pad 25: (no net) -> unconnected-(TEENSY_00-18_A4_SDA0-Pad25)
- TEENSY_00 pad 26: (no net) -> unconnected-(TEENSY_00-19_A5_SCL0-Pad26)
- TEENSY_00 pad 27: (no net) -> unconnected-(TEENSY_00-20_A6_TX5_LRCLK1-Pad27)
- TEENSY_00 pad 28: (no net) -> unconnected-(TEENSY_00-21_A7_RX5_BCLK1-Pad28)
- TEENSY_00 pad 3: (no net) -> unconnected-(TEENSY_00-1_TX1_CTX2_MISO1-Pad3)
- TEENSY_00 pad 34: (no net) -> unconnected-(TEENSY_00-VUSB-Pad34)
- TEENSY_00 pad 35: (no net) -> unconnected-(TEENSY_00-24_A10_TX6_SCL2-Pad35)
- TEENSY_00 pad 36: (no net) -> unconnected-(TEENSY_00-25_A11_RX6_SDA2-Pad36)
- TEENSY_00 pad 41: (no net) -> unconnected-(TEENSY_00-30_CRX3-Pad41)
- TEENSY_00 pad 42: (no net) -> unconnected-(TEENSY_00-31_CTX3-Pad42)
- TEENSY_00 pad 43: (no net) -> unconnected-(TEENSY_00-32_OUT1B-Pad43)
- TEENSY_00 pad 44: (no net) -> unconnected-(TEENSY_00-33_MCLK2-Pad44)
- TEENSY_00 pad 45: (no net) -> unconnected-(TEENSY_00-34_DAT1_MISO2-Pad45)
- TEENSY_00 pad 46: (no net) -> unconnected-(TEENSY_00-35_DAT0_MOSI2-Pad46)
- TEENSY_00 pad 48: (no net) -> unconnected-(TEENSY_00-36_CLK_CS2-Pad48)
- TEENSY_00 pad 49: (no net) -> unconnected-(TEENSY_00-3V3-Pad49)
- TEENSY_00 pad 50: (no net) -> unconnected-(TEENSY_00-37_CMD_SCK2-Pad50)
- TEENSY_00 pad 51: (no net) -> unconnected-(TEENSY_00-38_DAT3_RX5-Pad51)
- TEENSY_00 pad 52: (no net) -> unconnected-(TEENSY_00-39_DAT2_TX5-Pad52)
- TEENSY_00 pad 53: (no net) -> unconnected-(TEENSY_00-D--Pad53)
- TEENSY_00 pad 54: (no net) -> unconnected-(TEENSY_00-D+-Pad54)
Other:
- net class Default removed
